File: Myscion_Board_V1/Myscion_Board_V1.kicad_pcb (KiCad board)
At the start: 2 copper layers, 87 parts, among them SW1 1.0U_ESC, SW10 1.0U_8, SW11 1.0U_9, SW12 1.0U_0, SW13 1.0U_-, SW14 1.0U_=, SW15 2.0U_Back, SW16 1.5U_Tab, SW17 1.0U_Q, SW18 1.0U_W, SW19 1.0U_E, SW2 1.0U_~, SW20 1.0U_R, SW21 1.0U_T, SW22 1.0U_Y, SW23 1.0U_U, SW24 1.0U_I, SW25 1.0U_O, SW26 1.0U_P, SW27 1.0U_[, SW28 1.0U_], SW29 1.5U_\, SW3 1.0U_1, SW30 1.75U_CAPS, SW31 1.0U_A, SW32 1.0U_S, SW33 1.0U_D, SW34 1.0U_F, SW35 1.0U_G, SW36 1.0U_H, SW37 1.0U_J, SW38 1.0U_K, SW39 1.0U_L, SW4 1.0U_2, SW40 1.0U_:, SW41 1.0U_", SW42 2.25U_ENTER, SW43 2.25U_LSHIFT, SW44 1.0U_Z, SW45 1.0U_X, SW46 1.0U_C, SW47 1.0U_V, SW48 1.0U_B, SW49 1.0U_N, SW5 1.0U_3, SW50 1.0U_M, SW51 1.0U_<, SW52 1.0U_>, SW53 1.0U_?, SW54 2.75U_RSHIFT, SW55 1.25U_LCTRL, SW56 1.25U_LGUI, SW57 1.25U_LALT, SW58 6.25U_SPACE, SW59 1.25U_RALT, SW6 1.0U_4, SW60 1.25U_RGUI, SW61 1.25U_RMENU, SW62 1.25U_RCTRL, SW63 1.0U_F1, SW64 1.0U_F2, SW65 1.0U_4, SW66 1.0U_5, SW67 1.0U_2, SW68 1.0U_3, SW69 1.0U_4, SW7 1.0U_5, SW70 1.0U_5, SW71 1.0U_2, SW72 1.0U_3, SW73 1.0U_4, SW74 1.0U_5, SW75 ESC, SW76 F1, SW77 F2, SW78 F3, SW79 F4, SW8 1.0U_6, SW80 F5, SW81 F6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

Commit message: Keyboard Matrix complete
Parts:
- added REF**: D_DO-35_SOD27_P7.62mm_Horizontal, Diode_THT:D_DO-35_SOD27_P7.62mm_Horizontal, F.Cu at (350.0, 156.2)
- added REF**: D_SOD-123, Diode_SMD:D_SOD-123, F.Cu at (342.9, 161.9)
- added REF**: Nexperia_CFP3_SOD-123W, Diode_SMD:Nexperia_CFP3_SOD-123W, F.Cu at (350.0, 159.5)
- added REF**: R_MiniMELF_MMA-0204, Resistor_SMD:R_MiniMELF_MMA-0204, F.Cu at (354.8, 145.3)

Commit message: Key foot prints placed and locked down for the main keyboard
Parts:
- removed REF**: D_DO-35_SOD27_P7.62mm_Horizontal, Diode_THT:D_DO-35_SOD27_P7.62mm_Horizontal
- removed REF**: D_SOD-123, Diode_SMD:D_SOD-123
- removed REF**: Nexperia_CFP3_SOD-123W, Diode_SMD:Nexperia_CFP3_SOD-123W
- removed REF**: R_MiniMELF_MMA-0204, Resistor_SMD:R_MiniMELF_MMA-0204
- added D1: 75V, DB_SMD_Diodes:D_SOD-123, F.Cu at (276.9, 194.2)
- added D10: 75V, DB_SMD_Diodes:D_SOD-123, F.Cu at (294.3, 207.6)
- added D100: 75V, DB_SMD_Diodes:D_SOD-123, F.Cu at (282.7, 211.0)
- added D101: 75V, DB_SMD_Diodes:D_SOD-123, F.Cu at (282.7, 214.3)
- added D102: 75V, DB_SMD_Diodes:D_SOD-123, F.Cu at (288.5, 174.1)
- added D103: 75V, DB_SMD_Diodes:D_SOD-123, F.Cu at (288.5, 177.5)
- added D104: 75V, DB_SMD_Diodes:D_SOD-123, F.Cu at (288.5, 180.8)
- added D11: 75V, DB_SMD_Diodes:D_SOD-123, F.Cu at (294.3, 204.3)
- added D12: 75V, DB_SMD_Diodes:D_SOD-123, F.Cu at (294.3, 187.5)
- added D13: 75V, DB_SMD_Diodes:D_SOD-123, F.Cu at (288.5, 214.3)
- added D14: 75V, DB_SMD_Diodes:D_SOD-123, F.Cu at (288.5, 207.6)
- added D15: 75V, DB_SMD_Diodes:D_SOD-123, F.Cu at (288.5, 204.3)
- added D16: 75V, DB_SMD_Diodes:D_SOD-123, F.Cu at (288.5, 200.9)
- added D17: 75V, DB_SMD_Diodes:D_SOD-123, F.Cu at (317.4, 214.3)
- added D18: 75V, DB_SMD_Diodes:D_SOD-123, F.Cu at (276.9, 174.1)
- added D19: 75V, DB_SMD_Diodes:D_SOD-123, F.Cu at (276.9, 214.3)
- added D2: 75V, DB_SMD_Diodes:D_SOD-123, F.Cu at (317.4, 200.9)
- added D20: 75V, DB_SMD_Diodes:D_SOD-123, F.Cu at (282.7, 174.1)
- added D21: 75V, DB_SMD_Diodes:D_SOD-123, F.Cu at (317.4, 194.2)
- added D22: 75V, DB_SMD_Diodes:D_SOD-123, F.Cu at (317.4, 197.6)
- added D23: 75V, DB_SMD_Diodes:D_SOD-123, F.Cu at (317.4, 211.0)
- added D24: 75V, DB_SMD_Diodes:D_SOD-123, F.Cu at (311.6, 214.3)
- added D25: 75V, DB_SMD_Diodes:D_SOD-123, F.Cu at (311.6, 211.0)
- added D26: 75V, DB_SMD_Diodes:D_SOD-123, F.Cu at (311.6, 174.1)
- added D27: 75V, DB_SMD_Diodes:D_SOD-123, F.Cu at (305.8, 214.3)
- added D28: 75V, DB_SMD_Diodes:D_SOD-123, F.Cu at (305.8, 187.5)
- added D29: 75V, DB_SMD_Diodes:D_SOD-123, F.Cu at (305.8, 184.2)
- added D3: 75V, DB_SMD_Diodes:D_SOD-123, F.Cu at (317.4, 204.3)
- added D30: 75V, DB_SMD_Diodes:D_SOD-123, F.Cu at (305.8, 174.1)
- added D31: 75V, DB_SMD_Diodes:D_SOD-123, F.Cu at (294.3, 211.0)
- added D32: 75V, DB_SMD_Diodes:D_SOD-123, F.Cu at (294.3, 200.9)
- added D33: 75V, DB_SMD_Diodes:D_SOD-123, F.Cu at (294.3, 190.9)
- added D34: 75V, DB_SMD_Diodes:D_SOD-123, F.Cu at (294.3, 184.2)
- added D35: 75V, DB_SMD_Diodes:D_SOD-123, F.Cu at (294.3, 174.1)
- added D36: 75V, DB_SMD_Diodes:D_SOD-123, F.Cu at (288.5, 211.0)
- added D37: 75V, DB_SMD_Diodes:D_SOD-123, F.Cu at (288.5, 197.6)
- added D38: 75V, DB_SMD_Diodes:D_SOD-123, F.Cu at (276.9, 180.8)
- added D39: 75V, DB_SMD_Diodes:D_SOD-123, F.Cu at (276.9, 177.5)
- added D4: 75V, DB_SMD_Diodes:D_SOD-123, F.Cu at (317.4, 207.6)
- added D40: 75V, DB_SMD_Diodes:D_SOD-123, F.Cu at (276.9, 211.0)
- added D41: 75V, DB_SMD_Diodes:D_SOD-123, F.Cu at (317.4, 190.9)
- added D42: 75V, DB_SMD_Diodes:D_SOD-123, F.Cu at (317.4, 187.5)
- added D43: 75V, DB_SMD_Diodes:D_SOD-123, F.Cu at (317.4, 184.2)
- added D44: 75V, DB_SMD_Diodes:D_SOD-123, F.Cu at (317.4, 174.1)
- added D45: 75V, DB_SMD_Diodes:D_SOD-123, F.Cu at (311.6, 207.6)
- added D46: 75V, DB_SMD_Diodes:D_SOD-123, F.Cu at (311.6, 200.9)
- added D47: 75V, DB_SMD_Diodes:D_SOD-123, F.Cu at (305.8, 211.0)
- added D48: 75V, DB_SMD_Diodes:D_SOD-123, F.Cu at (305.8, 207.6)
- added D49: 75V, DB_SMD_Diodes:D_SOD-123, F.Cu at (305.8, 197.6)
- added D5: 75V, DB_SMD_Diodes:D_SOD-123, F.Cu at (311.6, 177.5)
- added D50: 75V, DB_SMD_Diodes:D_SOD-123, F.Cu at (300.1, 214.3)
- added D51: 75V, DB_SMD_Diodes:D_SOD-123, F.Cu at (294.3, 214.3)
- added D52: 75V, DB_SMD_Diodes:D_SOD-123, F.Cu at (294.3, 197.6)
- added D53: 75V, DB_SMD_Diodes:D_SOD-123, F.Cu at (294.3, 194.2)
- added D54: 75V, DB_SMD_Diodes:D_SOD-123, F.Cu at (294.3, 180.8)
- added D55: 75V, DB_SMD_Diodes:D_SOD-123, F.Cu at (294.3, 177.5)
- added D56: 75V, DB_SMD_Diodes:D_SOD-123, F.Cu at (288.5, 194.2)
- added D57: 75V, DB_SMD_Diodes:D_SOD-123, F.Cu at (288.5, 190.9)
- added D58: 75V, DB_SMD_Diodes:D_SOD-123, F.Cu at (276.9, 184.2)
- added D59: 75V, DB_SMD_Diodes:D_SOD-123, F.Cu at (276.9, 197.6)
- added D6: 75V, DB_SMD_Diodes:D_SOD-123, F.Cu at (305.8, 194.2)
- added D60: 75V, DB_SMD_Diodes:D_SOD-123, F.Cu at (276.9, 207.6)
- added D61: 75V, DB_SMD_Diodes:D_SOD-123, F.Cu at (282.7, 177.5)
- added D62: 75V, DB_SMD_Diodes:D_SOD-123, F.Cu at (317.4, 177.5)
- added D63: 75V, DB_SMD_Diodes:D_SOD-123, F.Cu at (311.6, 204.3)
- added D64: 75V, DB_SMD_Diodes:D_SOD-123, F.Cu at (311.6, 197.6)
- added D65: 75V, DB_SMD_Diodes:D_SOD-123, F.Cu at (311.6, 180.8)
- added D66: 75V, DB_SMD_Diodes:D_SOD-123, F.Cu at (305.8, 204.3)
- added D67: 75V, DB_SMD_Diodes:D_SOD-123, F.Cu at (305.8, 200.9)
- added D68: 75V, DB_SMD_Diodes:D_SOD-123, F.Cu at (300.1, 211.0)
- added D69: 75V, DB_SMD_Diodes:D_SOD-123, F.Cu at (300.1, 204.3)
- added D7: 75V, DB_SMD_Diodes:D_SOD-123, F.Cu at (305.8, 190.9)
- added D70: 75V, DB_SMD_Diodes:D_SOD-123, F.Cu at (300.1, 194.2)
- added D71: 75V, DB_SMD_Diodes:D_SOD-123, F.Cu at (300.1, 187.5)
- added D72: 75V, DB_SMD_Diodes:D_SOD-123, F.Cu at (300.1, 190.9)
- added D73: 75V, DB_SMD_Diodes:D_SOD-123, F.Cu at (300.1, 174.1)
- added D74: 75V, DB_SMD_Diodes:D_SOD-123, F.Cu at (288.5, 187.5)
- added D75: 75V, DB_SMD_Diodes:D_SOD-123, F.Cu at (276.9, 187.5)
- added D76: 75V, DB_SMD_Diodes:D_SOD-123, F.Cu at (276.9, 200.9)
- added D77: 75V, DB_SMD_Diodes:D_SOD-123, F.Cu at (276.9, 204.3)
- added D78: 75V, DB_SMD_Diodes:D_SOD-123, F.Cu at (282.7, 194.2)
- added D79: 75V, DB_SMD_Diodes:D_SOD-123, F.Cu at (317.4, 180.8)
- added D8: 75V, DB_SMD_Diodes:D_SOD-123, F.Cu at (305.8, 180.8)
- added D80: 75V, DB_SMD_Diodes:D_SOD-123, F.Cu at (311.6, 194.2)
- added D81: 75V, DB_SMD_Diodes:D_SOD-123, F.Cu at (311.6, 184.2)
- added D82: 75V, DB_SMD_Diodes:D_SOD-123, F.Cu at (311.6, 187.5)
- added D83: 75V, DB_SMD_Diodes:D_SOD-123, F.Cu at (311.6, 190.9)
- added D84: 75V, DB_SMD_Diodes:D_SOD-123, F.Cu at (300.1, 207.6)
- added D85: 75V, DB_SMD_Diodes:D_SOD-123, F.Cu at (300.1, 200.9)
- added D86: 75V, DB_SMD_Diodes:D_SOD-123, F.Cu at (300.1, 197.6)
- added D87: 75V, DB_SMD_Diodes:D_SOD-123, F.Cu at (300.1, 184.2)
- added D88: 75V, DB_SMD_Diodes:D_SOD-123, F.Cu at (300.1, 180.8)
- added D89: 75V, DB_SMD_Diodes:D_SOD-123, F.Cu at (300.1, 177.5)
- added D9: 75V, DB_SMD_Diodes:D_SOD-123, F.Cu at (305.8, 177.5)
- added D90: 75V, DB_SMD_Diodes:D_SOD-123, F.Cu at (288.5, 184.2)
- added D91: 75V, DB_SMD_Diodes:D_SOD-123, F.Cu at (276.9, 190.9)
- added D92: 75V, DB_SMD_Diodes:D_SOD-123, F.Cu at (282.7, 184.2)
- added D93: 75V, DB_SMD_Diodes:D_SOD-123, F.Cu at (282.7, 180.8)
- added D94: 75V, DB_SMD_Diodes:D_SOD-123, F.Cu at (282.7, 187.5)
- added D95: 75V, DB_SMD_Diodes:D_SOD-123, F.Cu at (282.7, 190.9)
- added D96: 75V, DB_SMD_Diodes:D_SOD-123, F.Cu at (282.7, 197.6)
- added D97: 75V, DB_SMD_Diodes:D_SOD-123, F.Cu at (282.7, 200.9)
- added D98: 75V, DB_SMD_Diodes:D_SOD-123, F.Cu at (282.7, 204.3)
- added D99: 75V, DB_SMD_Diodes:D_SOD-123, F.Cu at (282.7, 207.6)
- added SW100: Space, bk_Switch_Keyboard_Cherry_MX:SW_Cherry_MX_PCB_6.25u, F.Cu at (345.3, 152.4)
- added SW101: RightAlt, bk_Switch_Keyboard_Cherry_MX:SW_Cherry_MX_PCB_1.25u, F.Cu at (416.7, 152.4)
- added SW102: RightSystem, bk_Switch_Keyboard_Cherry_MX:SW_Cherry_MX_PCB_1.25u, F.Cu at (440.5, 152.4)
- added SW103: RightMenu, bk_Switch_Keyboard_Cherry_MX:SW_Cherry_MX_PCB_1.25u, F.Cu at (464.3, 152.4)
- added SW104: RightCtrl, bk_Switch_Keyboard_Cherry_MX:SW_Cherry_MX_PCB_1.25u, F.Cu at (488.2, 152.4)
- added SW88: >, bk_Switch_Keyboard_Cherry_MX:SW_Cherry_MX_PCB_1.00u, F.Cu at (419.1, 133.3)
- added SW89: ?, bk_Switch_Keyboard_Cherry_MX:SW_Cherry_MX_PCB_1.00u, F.Cu at (438.1, 133.3)
- added SW90: RightShift, bk_Switch_Keyboard_Cherry_MX:SW_Cherry_MX_PCB_2.75u, F.Cu at (473.9, 133.3)
- added SW91: Num0, bk_Switch_Keyboard_Cherry_MX:SW_Cherry_MX_PCB_2.00u, F.Cu at (85.7, 152.4)
- added SW92: Num., bk_Switch_Keyboard_Cherry_MX:SW_Cherry_MX_PCB_1.00u, F.Cu at (114.3, 152.4)
- added SW93: NumEnter, bk_Switch_Keyboard_Cherry_MX:SW_Cherry_MX_PCB_2.00u_90deg, F.Cu at (133.3, 142.9)
- added SW94: Left, bk_Switch_Keyboard_Cherry_MX:SW_Cherry_MX_PCB_1.00u, F.Cu at (159.5, 152.4)
- added SW95: Down, bk_Switch_Keyboard_Cherry_MX:SW_Cherry_MX_PCB_1.00u, F.Cu at (178.6, 152.4)
- added SW96: Right, bk_Switch_Keyboard_Cherry_MX:SW_Cherry_MX_PCB_1.00u, F.Cu at (197.6, 152.4)
- added SW97: LeftCtrl, bk_Switch_Keyboard_Cherry_MX:SW_Cherry_MX_PCB_1.25u, F.Cu at (226.2, 152.4)
- added SW98: LeftSystem, bk_Switch_Keyboard_Cherry_MX:SW_Cherry_MX_PCB_1.25u, F.Cu at (250.0, 152.4)
- added SW99: LeftAlt, bk_Switch_Keyboard_Cherry_MX:SW_Cherry_MX_PCB_1.25u, F.Cu at (273.8, 152.4)
- SW1: value 1.0U_ESC -> PrintScrn
- SW10: value 1.0U_8 -> F6
- SW11: value 1.0U_9 -> F7
- SW12: value 1.0U_0 -> F8
- SW13: value 1.0U_- -> F9
- SW14: value 1.0U_= -> F10
- SW15: value 2.0U_Back -> F11; footprint bk_Switch_Keyboard_Cherry_MX:SW_Cherry_MX_PCB_2.00u -> bk_Switch_Keyboard_Cherry_MX:SW_Cherry_MX_PCB_1.00u
- SW16: value 1.5U_Tab -> F12; footprint bk_Switch_Keyboard_Cherry_MX:SW_Cherry_MX_PCB_1.50u -> bk_Switch_Keyboard_Cherry_MX:SW_Cherry_MX_PCB_1.00u
- SW17: value 1.0U_Q -> NumPause
- SW18: value 1.0U_W -> Num/
- SW19: value 1.0U_E -> Num*
- SW2: value 1.0U_~ -> ScrollLk
- SW20: value 1.0U_R -> Num-
- SW21: value 1.0U_T -> Insert
- SW22: value 1.0U_Y -> Home
- SW23: value 1.0U_U -> PageUp
- SW24: value 1.0U_I -> Tilde
- SW25: value 1.0U_O -> 1
- SW26: value 1.0U_P -> 2
- SW27: value 1.0U_[ -> 3
- SW28: value 1.0U_] -> 4
- SW29: value 1.5U_\ -> 5; footprint bk_Switch_Keyboard_Cherry_MX:SW_Cherry_MX_PCB_1.50u -> bk_Switch_Keyboard_Cherry_MX:SW_Cherry_MX_PCB_1.00u
- SW3: value 1.0U_1 -> NumLk
- SW30: value 1.75U_CAPS -> 6; footprint bk_Switch_Keyboard_Cherry_MX:SW_Cherry_MX_PCB_1.75u -> bk_Switch_Keyboard_Cherry_MX:SW_Cherry_MX_PCB_1.00u
- SW31: value 1.0U_A -> 7
- SW32: value 1.0U_S -> 8
- SW33: value 1.0U_D -> 9
- SW34: value 1.0U_F -> 0
- SW35: value 1.0U_G -> -
- SW36: value 1.0U_H -> =
- SW37: value 1.0U_J -> Back; footprint bk_Switch_Keyboard_Cherry_MX:SW_Cherry_MX_PCB_1.00u -> bk_Switch_Keyboard_Cherry_MX:SW_Cherry_MX_PCB_2.00u
- SW38: value 1.0U_K -> Num7
- SW39: value 1.0U_L -> Num8
- SW4: value 1.0U_2 -> ESC
- SW40: value 1.0U_: -> Num9
- SW41: value 1.0U_" -> Delete
- SW42: value 2.25U_ENTER -> End; footprint bk_Switch_Keyboard_Cherry_MX:SW_Cherry_MX_PCB_2.25u -> bk_Switch_Keyboard_Cherry_MX:SW_Cherry_MX_PCB_1.00u
- SW43: value 2.25U_LSHIFT -> PageDown; footprint bk_Switch_Keyboard_Cherry_MX:SW_Cherry_MX_PCB_2.25u -> bk_Switch_Keyboard_Cherry_MX:SW_Cherry_MX_PCB_1.00u
- SW44: value 1.0U_Z -> Tab; footprint bk_Switch_Keyboard_Cherry_MX:SW_Cherry_MX_PCB_1.00u -> bk_Switch_Keyboard_Cherry_MX:SW_Cherry_MX_PCB_1.50u
- SW45: value 1.0U_X -> Q
- SW46: value 1.0U_C -> W
- SW47: value 1.0U_V -> E
- SW48: value 1.0U_B -> R
- SW49: value 1.0U_N -> T
- SW5: value 1.0U_3 -> F1
- SW50: value 1.0U_M -> Y
- SW51: value 1.0U_< -> U
- SW52: value 1.0U_> -> I
- SW53: value 1.0U_? -> O
- SW54: value 2.75U_RSHIFT -> P; footprint bk_Switch_Keyboard_Cherry_MX:SW_Cherry_MX_PCB_2.75u -> bk_Switch_Keyboard_Cherry_MX:SW_Cherry_MX_PCB_1.00u
- SW55: value 1.25U_LCTRL -> [; footprint bk_Switch_Keyboard_Cherry_MX:SW_Cherry_MX_PCB_1.25u -> bk_Switch_Keyboard_Cherry_MX:SW_Cherry_MX_PCB_1.00u
- SW56: value 1.25U_LGUI -> ]; footprint bk_Switch_Keyboard_Cherry_MX:SW_Cherry_MX_PCB_1.25u -> bk_Switch_Keyboard_Cherry_MX:SW_Cherry_MX_PCB_1.00u
- SW57: value 1.25U_LALT -> \; footprint bk_Switch_Keyboard_Cherry_MX:SW_Cherry_MX_PCB_1.25u -> bk_Switch_Keyboard_Cherry_MX:SW_Cherry_MX_PCB_1.50u
- SW58: value 6.25U_SPACE -> Num4; footprint bk_Switch_Keyboard_Cherry_MX:SW_Cherry_MX_PCB_6.25u -> bk_Switch_Keyboard_Cherry_MX:SW_Cherry_MX_PCB_1.00u
- SW59: value 1.25U_RALT -> Num5; footprint bk_Switch_Keyboard_Cherry_MX:SW_Cherry_MX_PCB_1.25u -> bk_Switch_Keyboard_Cherry_MX:SW_Cherry_MX_PCB_1.00u
- SW6: value 1.0U_4 -> F2
- SW60: value 1.25U_RGUI -> Num6; footprint bk_Switch_Keyboard_Cherry_MX:SW_Cherry_MX_PCB_1.25u -> bk_Switch_Keyboard_Cherry_MX:SW_Cherry_MX_PCB_1.00u
- SW61: value 1.25U_RMENU -> Num+; footprint bk_Switch_Keyboard_Cherry_MX:SW_Cherry_MX_PCB_1.25u -> bk_Switch_Keyboard_Cherry_MX:SW_Cherry_MX_PCB_2.00u_90deg
- SW62: value 1.25U_RCTRL -> CapsLk; footprint bk_Switch_Keyboard_Cherry_MX:SW_Cherry_MX_PCB_1.25u -> bk_Switch_Keyboard_Cherry_MX:SW_Cherry_MX_PCB_1.75u
- SW63: value 1.0U_F1 -> A
- SW64: value 1.0U_F2 -> S
- SW65: value 1.0U_4 -> D
- SW66: value 1.0U_5 -> F
- SW67: value 1.0U_2 -> G
- SW68: value 1.0U_3 -> H
- SW69: value 1.0U_4 -> J
- SW7: value 1.0U_5 -> F3
- SW70: value 1.0U_5 -> K
- SW71: value 1.0U_2 -> L
- SW72: value 1.0U_3 -> SemiColon
- SW73: value 1.0U_4 -> Quote
- SW74: value 1.0U_5 -> Enter; footprint bk_Switch_Keyboard_Cherry_MX:SW_Cherry_MX_PCB_1.00u -> bk_Switch_Keyboard_Cherry_MX:SW_Cherry_MX_PCB_2.25u
- SW75: value ESC -> Num1
- SW76: value F1 -> Num2
- SW77: value F2 -> Num3
- SW78: value F3 -> Up
- SW79: value F4 -> LeftShift; footprint bk_Switch_Keyboard_Cherry_MX:SW_Cherry_MX_PCB_1.00u -> bk_Switch_Keyboard_Cherry_MX:SW_Cherry_MX_PCB_2.25u
- SW8: value 1.0U_6 -> F4
- SW80: value F5 -> Z
- SW81: value F6 -> X
- SW82: value F7 -> C
- SW83: value F8 -> V
- SW84: value F9 -> B
- SW85: value F10 -> N
- SW86: value F11 -> M
- SW87: value F12 -> <
- SW9: value 1.0U_7 -> F5
- moved SW16 411.3 mm to (490.5, 57.1)
- moved SW87 375.3 mm to (400.1, 133.3)
- moved SW55 368.8 mm to (442.9, 95.2)
- moved SW56 364.1 mm to (462.0, 95.2)
- moved SW57 364.1 mm to (485.8, 95.2)
- moved SW84 349.0 mm to (342.9, 133.3)
- moved SW85 329.5 mm to (361.9, 133.3)
- moved SW83 325.0 mm to (323.9, 133.3)
- moved SW86 323.7 mm to (381.0, 133.3)
- moved SW82 301.2 mm to (304.8, 133.3)
- moved SW74 299.3 mm to (478.6, 114.3)
- moved SW72 295.5 mm to (428.6, 114.3)
- moved SW81 277.5 mm to (285.8, 133.3)
- moved SW71 271.0 mm to (409.6, 114.3)
- moved SW79 269.9 mm to (235.7, 133.3)
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Connections:
- SW1 pad 1: unconnected-(SW1-Pad1) -> Row0
- SW1 pad 2: unconnected-(SW1-Pad2) -> Net-(D1-K)
- SW10 pad 1: unconnected-(SW10-Pad1) -> Row0
- SW10 pad 2: unconnected-(SW10-Pad2) -> Net-(D10-K)
- SW11 pad 1: unconnected-(SW11-Pad1) -> Row0
- SW11 pad 2: unconnected-(SW11-Pad2) -> Net-(D11-K)
- SW12 pad 1: unconnected-(SW12-Pad1) -> Row0
- SW12 pad 2: unconnected-(SW12-Pad2) -> Net-(D12-K)
- SW13 pad 1: unconnected-(SW13-Pad1) -> Row0
- SW13 pad 2: unconnected-(SW13-Pad2) -> Net-(D13-K)
- SW14 pad 1: unconnected-(SW14-Pad1) -> Row0
- SW14 pad 2: unconnected-(SW14-Pad2) -> Net-(D14-K)
- SW15 pad 1: unconnected-(SW15-Pad1) -> Row0
- SW15 pad 2: unconnected-(SW15-Pad2) -> Net-(D15-K)
- SW16 pad 1: unconnected-(SW16-Pad1) -> Row0
- SW16 pad 2: unconnected-(SW16-Pad2) -> Net-(D16-K)
- SW17 pad 1: unconnected-(SW17-Pad1) -> Row1
- SW17 pad 2: unconnected-(SW17-Pad2) -> Net-(D17-K)
- SW18 pad 1: unconnected-(SW18-Pad1) -> Row1
- SW18 pad 2: unconnected-(SW18-Pad2) -> Net-(D18-K)
- SW19 pad 1: unconnected-(SW19-Pad1) -> Row1
- SW19 pad 2: unconnected-(SW19-Pad2) -> Net-(D19-K)
- SW2 pad 1: unconnected-(SW2-Pad1) -> Row0
- SW2 pad 2: unconnected-(SW2-Pad2) -> Net-(D2-K)
- SW20 pad 1: unconnected-(SW20-Pad1) -> Row1
- SW20 pad 2: unconnected-(SW20-Pad2) -> Net-(D20-K)
- SW21 pad 1: unconnected-(SW21-Pad1) -> Row1
- SW21 pad 2: unconnected-(SW21-Pad2) -> Net-(D21-K)
- SW22 pad 1: unconnected-(SW22-Pad1) -> Row1
- SW22 pad 2: unconnected-(SW22-Pad2) -> Net-(D22-K)
- SW23 pad 1: unconnected-(SW23-Pad1) -> Row1
- SW23 pad 2: unconnected-(SW23-Pad2) -> Net-(D23-K)
- SW24 pad 1: unconnected-(SW24-Pad1) -> Row1
- SW24 pad 2: unconnected-(SW24-Pad2) -> Net-(D24-K)
- SW25 pad 1: unconnected-(SW25-Pad1) -> Row1
- SW25 pad 2: unconnected-(SW25-Pad2) -> Net-(D25-K)
- SW26 pad 1: unconnected-(SW26-Pad1) -> Row1
- SW26 pad 2: unconnected-(SW26-Pad2) -> Net-(D26-K)
- SW27 pad 1: unconnected-(SW27-Pad1) -> Row1
- SW27 pad 2: unconnected-(SW27-Pad2) -> Net-(D27-K)
- SW28 pad 1: unconnected-(SW28-Pad1) -> Row1
- SW28 pad 2: unconnected-(SW28-Pad2) -> Net-(D28-K)
- SW29 pad 1: unconnected-(SW29-Pad1) -> Row1
- SW29 pad 2: unconnected-(SW29-Pad2) -> Net-(D29-K)
- SW3 pad 1: unconnected-(SW3-Pad1) -> Row0
- SW3 pad 2: unconnected-(SW3-Pad2) -> Net-(D3-K)
- SW30 pad 1: unconnected-(SW30-Pad1) -> Row1
- SW30 pad 2: unconnected-(SW30-Pad2) -> Net-(D30-K)
- SW31 pad 1: unconnected-(SW31-Pad1) -> Row1
- SW31 pad 2: unconnected-(SW31-Pad2) -> Net-(D31-K)
- SW32 pad 1: unconnected-(SW32-Pad1) -> Row1
- SW32 pad 2: unconnected-(SW32-Pad2) -> Net-(D32-K)
- SW33 pad 1: unconnected-(SW33-Pad1) -> Row1
- SW33 pad 2: unconnected-(SW33-Pad2) -> Net-(D33-K)
- SW34 pad 1: unconnected-(SW34-Pad1) -> Row1
- SW34 pad 2: unconnected-(SW34-Pad2) -> Net-(D34-K)
- SW35 pad 1: unconnected-(SW35-Pad1) -> Row1
- SW35 pad 2: unconnected-(SW35-Pad2) -> Net-(D35-K)
- SW36 pad 1: unconnected-(SW36-Pad1) -> Row1
- SW36 pad 2: unconnected-(SW36-Pad2) -> Net-(D36-K)
- SW37 pad 1: unconnected-(SW37-Pad1) -> Row1
- SW37 pad 2: unconnected-(SW37-Pad2) -> Net-(D37-K)
- SW38 pad 1: unconnected-(SW38-Pad1) -> Row2
- SW38 pad 2: unconnected-(SW38-Pad2) -> Net-(D38-K)
- SW39 pad 1: unconnected-(SW39-Pad1) -> Row2
- SW39 pad 2: unconnected-(SW39-Pad2) -> Net-(D39-K)
- SW4 pad 1: unconnected-(SW4-Pad1) -> Row0
- SW4 pad 2: unconnected-(SW4-Pad2) -> Net-(D4-K)
- SW40 pad 1: unconnected-(SW40-Pad1) -> Row2
- SW40 pad 2: unconnected-(SW40-Pad2) -> Net-(D40-K)
- SW41 pad 1: unconnected-(SW41-Pad1) -> Row2
- SW41 pad 2: unconnected-(SW41-Pad2) -> Net-(D41-K)
- SW42 pad 1: unconnected-(SW42-Pad1) -> Row2
- SW42 pad 2: unconnected-(SW42-Pad2) -> Net-(D42-K)
- SW43 pad 1: unconnected-(SW43-Pad1) -> Row2
- SW43 pad 2: unconnected-(SW43-Pad2) -> Net-(D43-K)
- SW44 pad 1: unconnected-(SW44-Pad1) -> Row2
- SW44 pad 2: unconnected-(SW44-Pad2) -> Net-(D44-K)
- SW45 pad 1: unconnected-(SW45-Pad1) -> Row2
- SW45 pad 2: unconnected-(SW45-Pad2) -> Net-(D45-K)
- SW46 pad 1: unconnected-(SW46-Pad1) -> Row2
- SW46 pad 2: unconnected-(SW46-Pad2) -> Net-(D46-K)
- SW47 pad 1: unconnected-(SW47-Pad1) -> Row2
- SW47 pad 2: unconnected-(SW47-Pad2) -> Net-(D47-K)
- SW48 pad 1: unconnected-(SW48-Pad1) -> Row2
- SW48 pad 2: unconnected-(SW48-Pad2) -> Net-(D48-K)
- SW49 pad 1: unconnected-(SW49-Pad1) -> Row2
- SW49 pad 2: unconnected-(SW49-Pad2) -> Net-(D49-K)
- SW5 pad 1: unconnected-(SW5-Pad1) -> Row0
- SW5 pad 2: unconnected-(SW5-Pad2) -> Net-(D5-K)
- SW50 pad 1: unconnected-(SW50-Pad1) -> Row2
- SW50 pad 2: unconnected-(SW50-Pad2) -> Net-(D50-K)
- SW51 pad 1: unconnected-(SW51-Pad1) -> Row2
- SW51 pad 2: unconnected-(SW51-Pad2) -> Net-(D51-K)
- SW52 pad 1: unconnected-(SW52-Pad1) -> Row2
- SW52 pad 2: unconnected-(SW52-Pad2) -> Net-(D52-K)
- SW53 pad 1: unconnected-(SW53-Pad1) -> Row2
- SW53 pad 2: unconnected-(SW53-Pad2) -> Net-(D53-K)
- SW54 pad 1: unconnected-(SW54-Pad1) -> Row2
- SW54 pad 2: unconnected-(SW54-Pad2) -> Net-(D54-K)
- SW55 pad 1: unconnected-(SW55-Pad1) -> Row2
- SW55 pad 2: unconnected-(SW55-Pad2) -> Net-(D55-K)
- SW56 pad 1: unconnected-(SW56-Pad1) -> Row2
- SW56 pad 2: unconnected-(SW56-Pad2) -> Net-(D56-K)
- SW57 pad 1: unconnected-(SW57-Pad1) -> Row2
- SW57 pad 2: unconnected-(SW57-Pad2) -> Net-(D57-K)
- SW58 pad 1: unconnected-(SW58-Pad1) -> Row3
- SW58 pad 2: unconnected-(SW58-Pad2) -> Net-(D58-K)
- SW59 pad 1: unconnected-(SW59-Pad1) -> Row3
- SW59 pad 2: unconnected-(SW59-Pad2) -> Net-(D59-K)
- SW6 pad 1: unconnected-(SW6-Pad1) -> Row0
- SW6 pad 2: unconnected-(SW6-Pad2) -> Net-(D6-K)
- SW60 pad 1: unconnected-(SW60-Pad1) -> Row3
- SW60 pad 2: unconnected-(SW60-Pad2) -> Net-(D60-K)
- SW61 pad 1: unconnected-(SW61-Pad1) -> Row3
- SW61 pad 2: unconnected-(SW61-Pad2) -> Net-(D61-K)
- SW62 pad 1: unconnected-(SW62-Pad1) -> Row3
- SW62 pad 2: unconnected-(SW62-Pad2) -> Net-(D62-K)
- SW63 pad 1: unconnected-(SW63-Pad1) -> Row3
- SW63 pad 2: unconnected-(SW63-Pad2) -> Net-(D63-K)
- SW64 pad 1: unconnected-(SW64-Pad1) -> Row3
- SW64 pad 2: unconnected-(SW64-Pad2) -> Net-(D64-K)
- SW65 pad 1: unconnected-(SW65-Pad1) -> Row3
- SW65 pad 2: unconnected-(SW65-Pad2) -> Net-(D65-K)
- SW66 pad 1: unconnected-(SW66-Pad1) -> Row3
- SW66 pad 2: unconnected-(SW66-Pad2) -> Net-(D66-K)
- SW67 pad 1: unconnected-(SW67-Pad1) -> Row3
- SW67 pad 2: unconnected-(SW67-Pad2) -> Net-(D67-K)
- SW68 pad 1: unconnected-(SW68-Pad1) -> Row3
- SW68 pad 2: unconnected-(SW68-Pad2) -> Net-(D68-K)
- SW69 pad 1: unconnected-(SW69-Pad1) -> Row3
- SW69 pad 2: unconnected-(SW69-Pad2) -> Net-(D69-K)
- SW7 pad 1: unconnected-(SW7-Pad1) -> Row0
- SW7 pad 2: unconnected-(SW7-Pad2) -> Net-(D7-K)
- SW70 pad 1: unconnected-(SW70-Pad1) -> Row3
- SW70 pad 2: unconnected-(SW70-Pad2) -> Net-(D70-K)
- SW71 pad 1: unconnected-(SW71-Pad1) -> Row3
- SW71 pad 2: unconnected-(SW71-Pad2) -> Net-(D71-K)
- SW72 pad 1: unconnected-(SW72-Pad1) -> Row3
- SW72 pad 2: unconnected-(SW72-Pad2) -> Net-(D72-K)
- SW73 pad 1: unconnected-(SW73-Pad1) -> Row3
- SW73 pad 2: unconnected-(SW73-Pad2) -> Net-(D73-K)
- SW74 pad 1: unconnected-(SW74-Pad1) -> Row3
- SW74 pad 2: unconnected-(SW74-Pad2) -> Net-(D74-K)
- SW75 pad 1: unconnected-(SW75-Pad1) -> Row4
- SW75 pad 2: unconnected-(SW75-Pad2) -> Net-(D75-K)
- SW76 pad 1: unconnected-(SW76-Pad1) -> Row4
- SW76 pad 2: unconnected-(SW76-Pad2) -> Net-(D76-K)
- SW77 pad 1: unconnected-(SW77-Pad1) -> Row4
- SW77 pad 2: unconnected-(SW77-Pad2) -> Net-(D77-K)
- SW78 pad 1: unconnected-(SW78-Pad1) -> Row4
- SW78 pad 2: unconnected-(SW78-Pad2) -> Net-(D78-K)
- SW79 pad 1: unconnected-(SW79-Pad1) -> Row4
- SW79 pad 2: unconnected-(SW79-Pad2) -> Net-(D79-K)
- SW8 pad 1: unconnected-(SW8-Pad1) -> Row0
- SW8 pad 2: unconnected-(SW8-Pad2) -> Net-(D8-K)
- SW80 pad 1: unconnected-(SW80-Pad1) -> Row4
- SW80 pad 2: unconnected-(SW80-Pad2) -> Net-(D80-K)
- SW81 pad 1: unconnected-(SW81-Pad1) -> Row4
- SW81 pad 2: unconnected-(SW81-Pad2) -> Net-(D81-K)
- SW82 pad 1: unconnected-(SW82-Pad1) -> Row4
- SW82 pad 2: unconnected-(SW82-Pad2) -> Net-(D82-K)
- SW83 pad 1: unconnected-(SW83-Pad1) -> Row4
- SW83 pad 2: unconnected-(SW83-Pad2) -> Net-(D83-K)
- SW84 pad 1: unconnected-(SW84-Pad1) -> Row4
- SW84 pad 2: unconnected-(SW84-Pad2) -> Net-(D84-K)
- SW85 pad 1: unconnected-(SW85-Pad1) -> Row4
- SW85 pad 2: unconnected-(SW85-Pad2) -> Net-(D85-K)
- SW86 pad 1: unconnected-(SW86-Pad1) -> Row4
- SW86 pad 2: unconnected-(SW86-Pad2) -> Net-(D86-K)
- SW87 pad 1: unconnected-(SW87-Pad1) -> Row4
- SW87 pad 2: unconnected-(SW87-Pad2) -> Net-(D87-K)
- SW9 pad 1: unconnected-(SW9-Pad1) -> Row0
- SW9 pad 2: unconnected-(SW9-Pad2) -> Net-(D9-K)
