File: Myscion_Board_V1/Myscion_Board_V1.kicad_sch (KiCad schematic)
At the start: 104 parts, among them SW1 Left, SW10 Num9, SW100 4, SW101 Back, SW102 Tab, SW103 T, SW104 Y, SW105 U, SW106 I, SW107 O, SW108 P, SW109 [, SW11 Num4, SW110 ], SW111 Q, SW112 W, SW113 E, SW114 R, SW115 \, SW116 PrintScrn, SW117 ScrollLk, SW118 NumLk, SW119 Insert, SW12 Num5, SW120 Home, SW121 PageUp, SW122 Delete, SW123 End, SW124 PageDown, SW125 CapsLk, SW126 G, SW127 H, SW128 J, SW129 K, SW13 Num6, SW130 L, SW131 :, SW132 ", SW133 A, SW134 S, SW135 D, SW136 F, SW137 Enter, SW138 LeftShift, SW139 B, SW14 Num1, SW140 N, SW141 M, SW142 <, SW143 >, SW144 ?, SW145 Z, SW146 X, SW147 C, SW148 V, SW149 RightShift, SW15 Num2, SW150 LeftCtrl, SW151 LeftSystem, SW152 LeftAlt, SW153 RightAlt, SW154 RightCtrl, SW155 RightSystem, SW156 RightMenu, SW157 Space, SW16 Num3, SW17 Num., SW18 Num0, SW19 Num-, SW2 Down, SW20 Num+, SW21 NumEnter, SW3 Right, SW4 Up, SW5 NumPause, SW6 Num/, SW7 Num*, SW75 ESC, SW76 F1, SW77 F2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

Commit message: Keyboard Matrix complete
Parts:
- removed SW115: \, bk_Switch_Keyboard_Cherry_MX:SW_Cherry_MX_PCB_1.50u, symbol DB:Mechanical_Keyboard/Cherry_MX_1.5U
- added D1, D10, D100, D101, D102, D103, D104, D11, D12, D13, D14, D15, D16, D17, D18, D19, D2, D20, D21, D22, D23, D24, D25, D26, D27, D28, D29, D3, D30, D31, D32, D33, D34, D35, D36, D37, D38, D39, D4, D40, D41, D42, D43, D44, D45, D46, D47, D48, D49, D5, D50, D51, D52, D53, D54, D55, D56, D57, D58, D59, D6, D60, D61, D62, D63, D64, D65, D66, D67, D68, D69, D7, D70, D71, D72, D73, D74, D75, D76, D77, D78, D79, D8, D80, D81, D82, D83, D84, D85, D86, D87, D88, D89, D9, D90, D91, D92, D93, D94, D95, D96, D97, D98, D99: 75V, DB_SMD_Diodes:D_SOD-123, symbol DB:Diode_SMD/Diode 75 V 150mA Surface Mount SOD-123
- added SW22: \, bk_Switch_Keyboard_Cherry_MX:SW_Cherry_MX_PCB_1.50u, symbol DB:Mechanical_Keyboard/Cherry_MX_1.5U
- SW131: value : -> SemiColon
- SW132: value " -> Quote
- SW96: value ~ -> Tilde
Connections:
- net Column21: now reaches SW149.1
- net Column21: now also SW101.1, SW137.1, SW154.1, SW87.1, SW22.1
- net at SW149.2: now also D42.2 (A)
- net Column15: now reaches SW91.1
- net Column15: now also SW106.1, SW129.1, SW141.1, SW82.1
- net at SW91.2: now also D86.2 (A)
- net Column14: now reaches SW128.1
- net Column14: now also SW105.1, SW140.1, SW81.1, SW90.1
- net at SW128.2: now also D58.2 (A)
- net at SW81.2: now also D32.2 (A)
- net Column8: now reaches SW111.1
- net Column8: now also SW133.1, SW151.1, SW97.1
- net at SW111.2: now also D70.2 (A)
- net Column19: now reaches SW95.1
- net Column19: now also SW85.1
- net at SW95.2: now also D82.2 (A)
- net Column3: now reaches SW19.1
- net Column3: now also SW20.1, SW21.1
- net at SW19.2: now also D4.2 (A)
- net at SW154.2: now also D43.2 (A)
- net Column7: now reaches SW138.1
- net Column7: now also SW102.1, SW125.1, SW150.1, SW75.1, SW96.1
- net at SW138.2: now also D51.2 (A)
- net Column10: now reaches SW113.1
- net Column10: now also SW135.1, SW146.1, SW77.1, SW99.1
- net at SW113.2: now also D72.2 (A)
- net Column9: now reaches SW134.1
- net Column9: now also SW112.1, SW145.1, SW152.1, SW76.1, SW98.1
- net at SW134.2: now also D63.2 (A)
- net at SW96.2: now also D104.2 (A)
- net Column12: now reaches SW103.1
- net Column12: now also SW126.1, SW148.1, SW79.1, SW88.1
- net at SW103.2: now also D74.2 (A)
- net Column0: now reaches SW8.1
- net Column0: now also SW11.1, SW14.1, SW18.1, SW5.1
- net at SW8.2: now also D5.2 (A)
- net Column18: now reaches SW132.1
- net Column18: now also SW109.1, SW144.1, SW155.1, SW84.1, SW94.1
- net at SW132.2: now also D99.2 (A)
- net at SW112.2: now also D71.2 (A)
- net Column6: now reaches SW121.1
- net Column6: now also SW118.1, SW124.1, SW3.1
- net at SW121.2: now also D103.2 (A)
- net at SW77.2: now also D28.2 (A)
- net at SW76.2: now also D27.2 (A)
- net at SW126.2: now also D60.2 (A)
- net at SW148.2: now also D55.2 (A)
- net Column13: now reaches SW127.1
- net Column13: now also SW104.1, SW139.1, SW157.1, SW80.1, SW89.1
- net at SW127.2: now also D59.2 (A)
- net Column2: now reaches SW17.1
- net Column2: now also SW16.1, SW7.1
- net at SW17.2: now also D15.2 (A)
- net at SW155.2: now also D45.2 (A)
- net at SW139.2: now also D56.2 (A)
- net Column16: now reaches SW92.1
- net Column16: now also SW107.1, SW130.1, SW142.1, SW83.1
- net at SW92.2: now also D85.2 (A)
- net at SW150.2: now also D50.2 (A)
- net at SW118.2: now also D25.2 (A)
- net at SW10.2: now also D7.2 (A)
- net at SW80.2: now also D31.2 (A)
- net at SW157.2: now also D47.2 (A)
- net Column17: now reaches SW108.1
- net Column17: now also SW131.1, SW143.1, SW153.1, SW93.1
- net at SW108.2: now also D79.2 (A)
- net Column20: now reaches SW156.1
- net Column20: now also SW110.1, SW86.1
- net at SW156.2: now also D44.2 (A)
- net at SW16.2: now also D11.2 (A)
- net at SW151.2: now also D49.2 (A)
- net Column5: now reaches SW4.1
- net Column5: now also SW117.1, SW120.1, SW123.1, SW2.1
- net at SW4.2: now also D24.2 (A)
- net at SW84.2: now also D35.2 (A)
- net at SW125.2: now also D65.2 (A)
- net at SW75.2: now also D26.2 (A)
- net Column11: now reaches SW78.1
- net Column11: now also SW100.1, SW114.1, SW136.1, SW147.1
- net at SW78.2: now also D29.2 (A)
- net at SW137.2: now also D41.2 (A)
- net at SW90.2: now also D87.2 (A)
- net at SW99.2: now also D91.2 (A)
- net at SW79.2: now also D30.2 (A)
- net Column4: now reaches SW119.1
- net Column4: now also SW1.1, SW116.1, SW122.1
- net at SW119.2: now also D19.2 (A)
- net at SW97.2: now also D93.2 (A)
- net at SW85.2: now also D36.2 (A)
- net at SW143.2: now also D97.2 (A)
- net at SW94.2: now also D83.2 (A)
- net at SW141.2: now also D95.2 (A)
- net at SW7.2: now also D3.2 (A)
- net at SW144.2: now also D98.2 (A)
- net at SW110.2: now also D81.2 (A)
- net at SW140.2: now also D57.2 (A)
- net at SW152.2: now also D48.2 (A)
- net at SW3.2: now also D23.2 (A)
- net at SW123.2: now also D67.2 (A)
- net at SW83.2: now also D34.2 (A)
- net at SW146.2: now also D53.2 (A)
- net at SW100.2: now also D90.2 (A)
- net at SW120.2: now also D102.2 (A)
- net at SW88.2: now also D89.2 (A)
- net Column1: now reaches SW12.1
- net Column1: now also SW15.1, SW6.1, SW9.1
- net at SW12.2: now also D9.2 (A)
- net at SW114.2: now also D73.2 (A)
- net at SW153.2: now also D46.2 (A)
- net at SW136.2: now also D61.2 (A)
- net at SW9.2: now also D6.2 (A)
- net at SW98.2: now also D92.2 (A)
- net at SW107.2: now also D78.2 (A)
- net at SW2.2: now also D22.2 (A)
- net at SW142.2: now also D96.2 (A)
- net at SW130.2: now also D101.2 (A)
- net at SW133.2: now also D64.2 (A)
- net at SW11.2: now also D8.2 (A)
- net at SW145.2: now also D52.2 (A)
- net at SW82.2: now also D33.2 (A)
- net at SW86.2: now also D37.2 (A)
- net at SW89.2: now also D88.2 (A)
- net at SW117.2: now also D20.2 (A)
- net at SW102.2: now also D69.2 (A)
- net at SW124.2: now also D68.2 (A)
- net at SW1.2: now also D21.2 (A)
- net at SW93.2: now also D84.2 (A)
- net at SW13.2: now also D10.2 (A)
- net at SW122.2: now also D66.2 (A)
- net at SW5.2: now also D1.2 (A)
- net at SW14.2: now also D13.2 (A)
- net at SW106.2: now also D77.2 (A)
- net at SW135.2: now also D62.2 (A)
- net at SW104.2: now also D75.2 (A)
- net at SW101.2: now also D39.2 (A)
- net at SW131.2: now also D100.2 (A)
- net at SW18.2: now also D14.2 (A)
- net at SW147.2: now also D54.2 (A)
- net at SW105.2: now also D76.2 (A)
- net at SW6.2: now also D2.2 (A)
- net at SW15.2: now also D12.2 (A)
- net at SW129.2: now also D94.2 (A)
- net at SW109.2: now also D80.2 (A)
- net at SW87.2: now also D38.2 (A)
- net at SW20.2: now also D17.2 (A)
- net at SW21.2: now also D16.2 (A)
- net at SW116.2: now also D18.2 (A)
- new net: D40.2 (A), SW22.2
- new net Row0: D18.1 (K), D20.1 (K), D25.1 (K), D26.1 (K), D27.1 (K), D28.1 (K), D29.1 (K), D30.1 (K), D31.1 (K), D32.1 (K), D33.1 (K), D34.1 (K), D35.1 (K), D36.1 (K), D37.1 (K), D38.1 (K)
- new net Row1: D1.1 (K), D102.1 (K), D103.1 (K), D104.1 (K), D19.1 (K), D2.1 (K), D3.1 (K), D39.1 (K), D4.1 (K), D82.1 (K), D83.1 (K), D84.1 (K), D85.1 (K), D86.1 (K), D87.1 (K), D88.1 (K), D89.1 (K), D90.1 (K), D91.1 (K), D92.1 (K), D93.1 (K)
- new net Row2: D40.1 (K), D5.1 (K), D6.1 (K), D66.1 (K), D67.1 (K), D68.1 (K), D69.1 (K), D7.1 (K), D70.1 (K), D71.1 (K), D72.1 (K), D73.1 (K), D74.1 (K), D75.1 (K), D76.1 (K), D77.1 (K), D78.1 (K), D79.1 (K), D80.1 (K), D81.1 (K)
- new net Row3: D10.1 (K), D100.1 (K), D101.1 (K), D17.1 (K), D41.1 (K), D58.1 (K), D59.1 (K), D60.1 (K), D61.1 (K), D62.1 (K), D63.1 (K), D64.1 (K), D65.1 (K), D8.1 (K), D9.1 (K), D94.1 (K), D99.1 (K)
- new net Row4: D11.1 (K), D12.1 (K), D13.1 (K), D24.1 (K), D42.1 (K), D51.1 (K), D52.1 (K), D53.1 (K), D54.1 (K), D55.1 (K), D56.1 (K), D57.1 (K), D95.1 (K), D96.1 (K), D97.1 (K), D98.1 (K)
- new net Row5: D14.1 (K), D15.1 (K), D16.1 (K), D21.1 (K), D22.1 (K), D23.1 (K), D43.1 (K), D44.1 (K), D45.1 (K), D46.1 (K), D47.1 (K), D48.1 (K), D49.1 (K), D50.1 (K)
Other:
- moved on the sheet: SW1, SW10, SW100, SW101, SW102, SW103, SW104, SW105, SW106, SW107, SW108, SW109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

Commit message: Moved diode to other side to aid in layout
Parts:
- removed D1: 75V, DB_SMD_Diodes:D_SOD-123, symbol DB:Diode_SMD/Diode 75 V 150mA Surface Mount SOD-123
- added D105: 75V, DB_SMD_Diodes:D_SOD-123, symbol DB:Diode_SMD/Diode 75 V 150mA Surface Mount SOD-123
Connections:
- net Column0: now also D4.2 (A), D5.2 (A), D6.2 (A), D7.2 (A), D105.2 (A); no longer SW11.1, SW14.1, SW18.1, SW5.1, SW8.1
- net Column1: now also D10.2 (A), D2.2 (A), D3.2 (A), D9.2 (A); no longer SW12.1, SW15.1, SW6.1, SW9.1
- net Column10: now also D73.2 (A), D78.2 (A), D79.2 (A), D82.2 (A), D83.2 (A); no longer SW113.1, SW135.1, SW146.1, SW77.1, SW99.1
- net Column11: now also D71.2 (A), D72.2 (A), D76.2 (A), D77.2 (A), D84.2 (A); no longer SW100.1, SW114.1, SW136.1, SW147.1, SW78.1
- net Column12: now also D69.2 (A), D70.2 (A), D74.2 (A), D75.2 (A), D85.2 (A); no longer SW103.1, SW126.1, SW148.1, SW79.1, SW88.1
- net Column13: now also D26.2 (A), D64.2 (A), D65.2 (A), D66.2 (A), D67.2 (A), D68.2 (A); no longer SW104.1, SW127.1, SW139.1, SW157.1, SW80.1, SW89.1
- net Column14: now also D51.2 (A), D52.2 (A), D53.2 (A), D62.2 (A), D63.2 (A); no longer SW105.1, SW128.1, SW140.1, SW81.1, SW90.1
- net Column15: now also D48.2 (A), D49.2 (A), D50.2 (A), D60.2 (A), D61.2 (A); no longer SW106.1, SW129.1, SW141.1, SW82.1, SW91.1
- net Column16: now also D45.2 (A), D46.2 (A), D47.2 (A), D57.2 (A), D58.2 (A); no longer SW107.1, SW130.1, SW142.1, SW83.1, SW92.1
- net Column17: now also D27.2 (A), D43.2 (A), D44.2 (A), D56.2 (A), D59.2 (A); no longer SW108.1, SW131.1, SW143.1, SW153.1, SW93.1
- net Column18: now also D28.2 (A), D40.2 (A), D41.2 (A), D42.2 (A), D54.2 (A), D55.2 (A); no longer SW109.1, SW132.1, SW144.1, SW155.1, SW84.1, SW94.1
- net Column19: now also D38.2 (A), D39.2 (A); no longer SW85.1, SW95.1
- net Column2: now also D11.2 (A), D12.2 (A), D13.2 (A), D14.2 (A), D18.2 (A); no longer SW16.1, SW17.1, SW7.1
- net Column20: now also D29.2 (A), D34.2 (A), D37.2 (A); no longer SW110.1, SW156.1, SW86.1
- net Column21: now also D30.2 (A), D31.2 (A), D32.2 (A), D33.2 (A), D35.2 (A), D36.2 (A); no longer SW101.1, SW137.1, SW149.1, SW154.1, SW22.1, SW87.1
- net Column3: now also D15.2 (A), D16.2 (A), D17.2 (A); no longer SW19.1, SW20.1, SW21.1
- net Column4: now also D19.2 (A), D8.2 (A), D98.2 (A), D99.2 (A); no longer SW1.1, SW116.1, SW119.1, SW122.1
- net Column5: now also D100.2 (A), D101.2 (A), D20.2 (A), D21.2 (A), D97.2 (A); no longer SW117.1, SW120.1, SW123.1, SW2.1, SW4.1
- net Column6: now also D102.2 (A), D104.2 (A), D22.2 (A), D96.2 (A); no longer SW118.1, SW121.1, SW124.1, SW3.1
- net Column7: now also D103.2 (A), D23.2 (A), D92.2 (A), D93.2 (A), D94.2 (A), D95.2 (A); no longer SW102.1, SW125.1, SW138.1, SW150.1, SW75.1, SW96.1
- net Column8: now also D24.2 (A), D89.2 (A), D90.2 (A), D91.2 (A); no longer SW111.1, SW133.1, SW151.1, SW97.1
- net Column9: now also D25.2 (A), D80.2 (A), D81.2 (A), D86.2 (A), D87.2 (A), D88.2 (A); no longer SW112.1, SW134.1, SW145.1, SW152.1, SW76.1, SW98.1
- net Row0: now also SW116.1, SW117.1, SW118.1, SW75.1, SW76.1, SW77.1, SW78.1, SW79.1, SW80.1, SW81.1, SW82.1, SW83.1, SW84.1, SW85.1, SW86.1, SW87.1; no longer D18.1 (K), D20.1 (K), D25.1 (K), D26.1 (K), D27.1 (K), D28.1 (K), D29.1 (K), D30.1 (K), D31.1 (K), D32.1 (K), D33.1 (K), D34.1 (K), D35.1 (K), D36.1 (K), D37.1 (K), D38.1 (K)
- net Row1: now also SW100.1, SW101.1, SW119.1, SW120.1, SW121.1, SW19.1, SW5.1, SW6.1, SW7.1, SW88.1, SW89.1, SW90.1, SW91.1, SW92.1, SW93.1, SW94.1, SW95.1, SW96.1, SW97.1, SW98.1, SW99.1; no longer D102.1 (K), D103.1 (K), D104.1 (K), D19.1 (K), D2.1 (K), D3.1 (K), D39.1 (K), D4.1 (K), D82.1 (K), D83.1 (K), D84.1 (K), D85.1 (K), D86.1 (K), D87.1 (K), D88.1 (K), D89.1 (K), D90.1 (K), D91.1 (K), D92.1 (K), D93.1 (K)
- net Row2: now also SW10.1, SW102.1, SW103.1, SW104.1, SW105.1, SW106.1, SW107.1, SW108.1, SW109.1, SW110.1, SW111.1, SW112.1, SW113.1, SW114.1, SW122.1, SW123.1, SW124.1, SW22.1, SW8.1, SW9.1; no longer D40.1 (K), D5.1 (K), D6.1 (K), D66.1 (K), D67.1 (K), D68.1 (K), D69.1 (K), D7.1 (K), D70.1 (K), D71.1 (K), D72.1 (K), D73.1 (K), D74.1 (K), D75.1 (K), D76.1 (K), D77.1 (K), D78.1 (K), D79.1 (K), D80.1 (K), D81.1 (K)
- net Row3: now also SW11.1, SW12.1, SW125.1, SW126.1, SW127.1, SW128.1, SW129.1, SW13.1, SW130.1, SW131.1, SW132.1, SW133.1, SW134.1, SW135.1, SW136.1, SW137.1, SW20.1; no longer D10.1 (K), D100.1 (K), D101.1 (K), D17.1 (K), D41.1 (K), D58.1 (K), D59.1 (K), D60.1 (K), D61.1 (K), D62.1 (K), D63.1 (K), D64.1 (K), D65.1 (K), D8.1 (K), D9.1 (K), D94.1 (K), D99.1 (K)
- net Row4: now also SW138.1, SW139.1, SW14.1, SW140.1, SW141.1, SW142.1, SW143.1, SW144.1, SW145.1, SW146.1, SW147.1, SW148.1, SW149.1, SW15.1, SW16.1, SW4.1; no longer D11.1 (K), D12.1 (K), D13.1 (K), D24.1 (K), D42.1 (K), D51.1 (K), D52.1 (K), D53.1 (K), D54.1 (K), D55.1 (K), D56.1 (K), D57.1 (K), D95.1 (K), D96.1 (K), D97.1 (K), D98.1 (K)
- net Row5: now also SW1.1, SW150.1, SW151.1, SW152.1, SW153.1, SW154.1, SW155.1, SW156.1, SW157.1, SW17.1, SW18.1, SW2.1, SW21.1, SW3.1; no longer D14.1 (K), D15.1 (K), D16.1 (K), D21.1 (K), D22.1 (K), D23.1 (K), D43.1 (K), D44.1 (K), D45.1 (K), D46.1 (K), D47.1 (K), D48.1 (K), D49.1 (K), D50.1 (K)
- net at SW149.2: now also D31.1 (K); no longer D42.2 (A)
- net at SW151.2: now also D24.1 (K); no longer D49.2 (A)
- net at SW98.2: now also D80.1 (K); no longer D92.2 (A)
- net at SW91.2: now also D49.1 (K); no longer D86.2 (A)
- net at SW128.2: now also D63.1 (K); no longer D58.2 (A)
- net at SW81.2: now also D51.1 (K); no longer D32.2 (A)
- net at SW111.2: now also D90.1 (K); no longer D70.2 (A)
- net at SW122.2: now also D98.1 (K); no longer D66.2 (A)
- net at SW13.2: now also D12.1 (K); no longer D10.2 (A)
- net at SW95.2: now also D39.1 (K); no longer D82.2 (A)
- net at SW19.2: now also D15.1 (K); no longer D4.2 (A)
- net at SW154.2: now also D30.1 (K); no longer D43.2 (A)
- net at SW138.2: now also D95.1 (K); no longer D51.2 (A)
- net at SW17.2: now also D18.1 (K); no longer D15.2 (A)
- net at SW113.2: now also D78.1 (K); no longer D72.2 (A)
- net at SW134.2: now also D87.1 (K); no longer D63.2 (A)
- net at SW156.2: now also D29.1 (K); no longer D44.2 (A)
- net at SW124.2: now also D96.1 (K); no longer D68.2 (A)
- net at SW5.2: now also D105.1 (K)
- net at SW96.2: now also D92.1 (K); no longer D104.2 (A)
- net at SW103.2: now also D74.1 (K); no longer D74.2 (A)
- net at SW118.2: now also D102.1 (K); no longer D25.2 (A)
- net at SW90.2: now also D52.1 (K); no longer D87.2 (A)
- net at SW8.2: now also D4.1 (K); no longer D5.2 (A)
- net at SW4.2: now also D21.1 (K); no longer D24.2 (A)
- net at SW132.2: now also D54.1 (K); no longer D99.2 (A)
- net at SW86.2: now also D37.1 (K); no longer D37.2 (A)
- net at SW152.2: now also D25.1 (K); no longer D48.2 (A)
- net at SW112.2: now also D88.1 (K); no longer D71.2 (A)
- net at SW101.2: now also D35.1 (K); no longer D39.2 (A)
- net at SW121.2: now also D104.1 (K); no longer D103.2 (A)
- net at SW150.2: now also D23.1 (K); no longer D50.2 (A)
- net at SW116.2: now also D8.1 (K); no longer D18.2 (A)
- net at SW10.2: now also D13.1 (K); no longer D7.2 (A)
- net at SW77.2: now also D73.1 (K); no longer D28.2 (A)
- net at SW14.2: now also D6.1 (K); no longer D13.2 (A)
- net at SW76.2: now also D81.1 (K); no longer D27.2 (A)
- net at SW12.2: now also D9.1 (K); no longer D9.2 (A)
- net at SW126.2: now also D75.1 (K); no longer D60.2 (A)
- net at SW148.2: now also D85.1 (K); no longer D55.2 (A)
- net at SW127.2: now also D65.1 (K); no longer D59.2 (A)
- net at SW139.2: now also D64.1 (K); no longer D56.2 (A)
- net at SW144.2: now also D55.1 (K); no longer D98.2 (A)
- net at SW114.2: now also D77.1 (K); no longer D73.2 (A)
- net at SW107.2: now also D47.1 (K); no longer D78.2 (A)
- net at SW123.2: now also D97.1 (K); no longer D67.2 (A)
- net at SW155.2: now also D28.1 (K); no longer D45.2 (A)
- net at SW92.2: now also D46.1 (K); no longer D85.2 (A)
- net at SW102.2: now also D93.1 (K); no longer D69.2 (A)
- net at SW136.2: now also D76.1 (K); no longer D61.2 (A)
- net at SW125.2: now also D94.1 (K); no longer D65.2 (A)
- net at SW80.2: now also D68.1 (K); no longer D31.2 (A)
- net at SW157.2: now also D26.1 (K); no longer D47.2 (A)
- net at SW108.2: now also D43.1 (K); no longer D79.2 (A)
- net at SW153.2: now also D27.1 (K); no longer D46.2 (A)
- net at SW88.2: now also D70.1 (K); no longer D89.2 (A)
- net at SW119.2: now also D99.1 (K); no longer D19.2 (A)
- net at SW16.2: now also D11.1 (K); no longer D11.2 (A)
- net at SW20.2: now also D16.1 (K); no longer D17.2 (A)
- net at SW84.2: now also D40.1 (K); no longer D35.2 (A)
- net at SW130.2: now also D58.1 (K); no longer D101.2 (A)
- net at SW75.2: now also D103.1 (K); no longer D26.2 (A)
- net at SW147.2: now also D84.1 (K); no longer D54.2 (A)
- net at SW78.2: now also D72.1 (K); no longer D29.2 (A)
- net at SW137.2: now also D32.1 (K); no longer D41.2 (A)
- net at SW145.2: now also D86.1 (K); no longer D52.2 (A)
- net at SW18.2: now also D7.1 (K); no longer D14.2 (A)
- net at SW79.2: now also D69.1 (K); no longer D30.2 (A)
- net at SW99.2: now also D79.1 (K); no longer D91.2 (A)
- net at SW142.2: now also D57.1 (K); no longer D96.2 (A)
- net at SW97.2: now also D91.1 (K); no longer D93.2 (A)
- net at SW85.2: now also D38.1 (K); no longer D36.2 (A)
- net at SW143.2: now also D56.1 (K); no longer D97.2 (A)
- net at SW105.2: now also D53.1 (K); no longer D76.2 (A)
- net at SW94.2: now also D41.1 (K); no longer D83.2 (A)
- net at SW110.2: now also D34.1 (K); no longer D81.2 (A)
- net at SW141.2: now also D61.1 (K); no longer D95.2 (A)
- net at SW9.2: now also D3.1 (K); no longer D6.2 (A)
- net at SW131.2: now also D59.1 (K); no longer D100.2 (A)
- net at SW146.2: now also D83.1 (K); no longer D53.2 (A)
- net at SW7.2: now also D14.1 (K); no longer D3.2 (A)
- net at SW1.2: now also D19.1 (K); no longer D21.2 (A)
- net at SW140.2: now also D62.1 (K); no longer D57.2 (A)
- net at SW3.2: now also D22.1 (K); no longer D23.2 (A)
- net at SW129.2: now also D60.1 (K); no longer D94.2 (A)
- net at SW83.2: now also D45.1 (K); no longer D34.2 (A)
- net at SW100.2: now also D71.1 (K); no longer D90.2 (A)
- net at SW120.2: now also D100.1 (K); no longer D102.2 (A)
- net at SW109.2: now also D42.1 (K); no longer D80.2 (A)
- net at SW135.2: now also D82.1 (K); no longer D62.2 (A)
- net at SW22.2: now also D33.1 (K); no longer D40.2 (A)
- net at SW2.2: now also D20.1 (K); no longer D22.2 (A)
- net at SW93.2: now also D44.1 (K); no longer D84.2 (A)
- net at SW87.2: now also D36.1 (K); no longer D38.2 (A)
- net at SW15.2: now also D10.1 (K); no longer D12.2 (A)
- net at SW133.2: now also D89.1 (K); no longer D64.2 (A)
- net at SW106.2: now also D48.1 (K); no longer D77.2 (A)
- net at SW11.2: now also D5.1 (K); no longer D8.2 (A)
- net at SW82.2: now also D50.1 (K); no longer D33.2 (A)
- net at SW117.2: now also D101.1 (K); no longer D20.2 (A)
- net at SW89.2: now also D67.1 (K); no longer D88.2 (A)
- net at SW21.2: now also D17.1 (K); no longer D16.2 (A)
- net at SW104.2: now also D66.1 (K); no longer D75.2 (A)
- net at SW6.2: now also D2.1 (K); no longer D2.2 (A)
Other:
- moved on the sheet: SW1, SW10, SW100, SW101, SW102, SW103, SW104, SW105, SW106, SW107, SW108, SW109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

Commit message: Key foot prints placed and locked down for the main keyboard
Parts:
- renumbered D8 to D1, D51 to D10, D26 to D100, D27 to D101, D28 to D102, D29 to D103, D30 to D104, D50 to D11, D45 to D12, D40 to D13, D38 to D14, D37 to D15, D36 to D16, D105 to D17, D2 to D18, D14 to D19, D101 to D2, D15 to D20, D99 to D21, D100 to D22, D104 to D23, D92 to D24, D91 to D25, D80 to D26, D79 to D27, D71 to D28, D70 to D29, D102 to D3, D67 to D30, D52 to D31, D49 to D32, D46 to D33, D44 to D34, D41 to D35, D39 to D36, D35 to D37, D4 to D38, D3 to D39, D103 to D4, D13 to D40, D98 to D41, D97 to D42, D96 to D43, D93 to D44, D90 to D45, D88 to D46, D78 to D47, D77 to D48, D74 to D49, D81 to D5, D66 to D50, D53 to D51, D48 to D52, D47 to D53, D43 to D54, D42 to D55, D34 to D56, D33 to D57, D5 to D58, D9 to D59, D73 to D6, D12 to D60, D16 to D61, D94 to D62, D89 to D63, D87 to D64, D82 to D65, D76 to D66, D75 to D67, D65 to D68, D63 to D69, D72 to D7, D60 to D70, D58 to D71, D59 to D72, D54 to D73, D32 to D74, D6 to D75, D10 to D76, D11 to D77, D21 to D78, D95 to D79, D69 to D8, D86 to D80, D83 to D81, D84 to D82, D85 to D83, D64 to D84, D62 to D85, D61 to D86, D57 to D87, D56 to D88, D55 to D89, D68 to D9, D31 to D90, D7 to D91, D18 to D92, D17 to D93, D19 to D94, D20 to D95, D22 to D96, D23 to D97, D24 to D98, D25 to D99, SW116 to SW1, SW81 to SW10, SW157 to SW100, SW153 to SW101, SW155 to SW102, SW156 to SW103, SW154 to SW104, SW82 to SW11, SW83 to SW12, SW84 to SW13, SW85 to SW14, SW86 to SW15, SW87 to SW16, SW5 to SW17, SW6 to SW18, SW7 to SW19, SW117 to SW2, SW19 to SW20, SW119 to SW21, SW120 to SW22, SW121 to SW23, SW96 to SW24, SW97 to SW25, SW98 to SW26, SW99 to SW27, SW100 to SW28, SW88 to SW29, SW118 to SW3, SW89 to SW30, SW90 to SW31, SW91 to SW32, SW92 to SW33, SW93 to SW34, SW94 to SW35, SW95 to SW36, SW101 to SW37, SW8 to SW38, SW9 to SW39, SW75 to SW4, SW10 to SW40, SW122 to SW41, SW123 to SW42, SW124 to SW43, SW102 to SW44, SW111 to SW45, SW112 to SW46, SW113 to SW47, SW114 to SW48, SW103 to SW49, SW76 to SW5, SW104 to SW50, SW105 to SW51, SW106 to SW52, SW107 to SW53, SW108 to SW54, SW109 to SW55, SW110 to SW56, SW22 to SW57, SW11 to SW58, SW12 to SW59, SW77 to SW6, SW13 to SW60, SW20 to SW61, SW125 to SW62, SW133 to SW63, SW134 to SW64, SW135 to SW65, SW136 to SW66, SW126 to SW67, SW127 to SW68, SW128 to SW69, SW78 to SW7, SW129 to SW70, SW130 to SW71, SW131 to SW72, SW132 to SW73, SW137 to SW74, SW14 to SW75, SW15 to SW76, SW16 to SW77, SW4 to SW78, SW138 to SW79, SW79 to SW8, SW145 to SW80, SW146 to SW81, SW147 to SW82, SW148 to SW83, SW139 to SW84, SW140 to SW85, SW141 to SW86, SW142 to SW87, SW143 to SW88, SW144 to SW89, SW80 to SW9, SW149 to SW90, SW18 to SW91, SW17 to SW92, SW21 to SW93, SW1 to SW94, SW2 to SW95, SW3 to SW96, SW150 to SW97, SW151 to SW98, SW152 to SW99
Other:
- note added: "Myscion Dynamics"
